Commit message: Edit model description

File: crab_description/models/crab_leg.xacro (robot description, xacro)
@@ -19,6 +19,5 @@
     		</visual>
 	</link>
-<!-- Pi parameter -->
-	<xacro:property name="pi" value="3.1415926535897931" />
+<!-- Pi is already defined: http://wiki.ros.org/xacro#Math_expressions -->
 <!-- Joint properties -->
 	<xacro:property name="joint_lower_limit" value="-${pi/2}" />

File: crab_description/models/crab_model.xacro (robot description, xacro)
@@ -19,6 +19,4 @@
     		</visual>
 	</link>
-<!-- Pi parameter -->
-	<xacro:property name="pi" value="3.1415926535897931" />
 <!-- Joint properties -->
 	<xacro:property name="joint_lower_limit" value="-${1.5}" />
